File: single_ended_differential_converter.sch (KiCad schematic (older format))
At the start: 27 parts, among them J1 Conn_Coaxial, J2 Conn_Coaxial, J5 XLR3, U1 PWR_JACK_POS, U2 PWR_JACK_GND, U3 PWR_JACK_NEG, U4 ADA4941-1

Commit message: added files for version 2
Parts:
- removed U3: PWR_JACK_NEG, Connector:Banana_Jack_1Pin, symbol my_library:PWR_JACK_NEG
- removed U4: ADA4941-1, Package_SO:SOIC-8-N7_3.9x4.9mm_P1.27mm, symbol my_library:ADA4941-1
- added C4, C5: C, Capacitor_SMD:C_0805_2012Metric_Pad1.15x1.40mm_HandSolder, symbol Device:C
- added CF2: 100pF, Capacitor_SMD:C_0805_2012Metric_Pad1.15x1.40mm_HandSolder, symbol Device:C
- added R10, R9, RO1, RO2: R_US, Resistor_SMD:R_0805_2012Metric_Pad1.15x1.40mm_HandSolder, symbol Device:R_US
- added R8, RF2: 10k, Resistor_SMD:R_0805_2012Metric_Pad1.15x1.40mm_HandSolder, symbol Device:R_US
- added TP1: OUTi-, my_library_foot:TestPoint_Keystone_5000-5004_Miniature, symbol Connector:TestPoint
- added TP2: OUTi+, my_library_foot:TestPoint_Keystone_5000-5004_Miniature, symbol Connector:TestPoint
- added TP3: VINV1, my_library_foot:TestPoint_Keystone_5000-5004_Miniature, symbol Connector:TestPoint
- added TP4: VINV2, my_library_foot:TestPoint_Keystone_5000-5004_Miniature, symbol Connector:TestPoint
- added U3, U4: OPA376xxDBV, Package_TO_SOT_SMD:SOT-23-5, symbol Amplifier_Operational:OPA376xxDBV
- C3: value 100uF -> 10uF; footprint Capacitor_SMD:CP_Elec_8x10 -> Capacitor_SMD:C_0805_2012Metric_Pad1.15x1.40mm_HandSolder
- CF1: value ? -> 100pF
- R5: value 10k -> 30k
- VOS1: value TestPoint -> VOS1
- VOS2: value TestPoint -> VOS2
Connections:
- net labels added: COMP1, COMP2, INV1, INV2, OUT+, OUT-, OUTi+, OUTi-
- net labels removed: VSS, VoutN, VoutP
- wire segments 58 -> 81
Other:
- moved on the sheet: C1, H1, H2, H3, H4
